Commit message: added changed files

File: urdf/sherpa_busy_genius.urdf (robot description, URDF)
Before this commit: robot busy_genius, 70 links, 69 joints
Links:
- link left_toe_z: geometry collision mesh filename=package://sherpa_spatial_relations/meshes/ToeLeft.dae.stl; visual mesh filename=package://sherpa_spatial_relations/meshes/ToeLeft.dae

Commit message: added all stuff

File: urdf/sherpa_busy_genius.urdf (robot description, URDF)
Before this commit: robot /, 70 links, 69 joints
Links:
- added link hand_laser_box_link, mass 0.01; collision box size=0.05 0.05 0.1; visual box size=0.05 0.05 0.1
Joints:
- added joint side_laser_box_joint: type fixed, parent hand_laser_link, child hand_laser_box_link, origin xyz=0 0 0 rpy=0 0 0

Commit message: added new files and genius

File: urdf/sherpa_busy_genius.urdf (robot description, URDF)
Before this commit: robot /, 71 links, 70 joints
Links:
- removed link hand_laser_box_link
- added link camera_depth_frame
- added link camera_depth_optical_frame
- added link camera_link, mass 0.001; collision mesh filename=package://hector_sensors_description/meshes/kinect_camera/k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; visual mesh filename=package://sherpa_spatial_relations/meshes/hokuyo.dae
- added link camera_rgb_frame
- added link camera_rgb_optical_frame
Joints:
- removed joint side_laser_box_joint
- added joint camera_depth_joint: type fixed, parent camera_link, child camera_depth_frame, origin xyz=0.0 -0.02 0.0 rpy=0 0 0
- added joint camera_depth_optical_joint: type fixed, parent camera_depth_frame, child camera_depth_optical_frame, origin xyz=0 0 0 rpy=-1.57079632679 0.0 -1.57079632679
- added joint camera_joint: type fixed, parent right_hand_y, child camera_link, origin xyz=-0.01 0 0 rpy=0 0 1.5
- added joint camera_rgb_joint: type fixed, parent camera_link, child camera_rgb_frame, origin xyz=0.0 -0.0125 0.0 rpy=0 0 0
- added joint camera_rgb_optical_joint: type fixed, parent camera_rgb_frame, child camera_rgb_optical_frame, origin xyz=0 0 0 rpy=-1.57079632679 0.0 -1.57079632679

File: urdf/tree-4.urdf (robot description, URDF)
Before this commit: robot tree1, 1 links, 0 joints
Links:
- link base_link: geometry collision mesh filename=package://sherpa_spatial_relations/models/tree-4.stl; visual mesh filename=package://sherpa_spatial_relations/meshes/tree-4.dae

Commit message: added all stuff

File: urdf/sherpa_busy_genius.urdf (robot description, URDF)
Before this commit: robot /, 75 links, 74 joints
Links:
- link camera_link: geometry collision mesh filename=package://sherpa_spatial_relations/meshes/hokuyo.dae; visual mesh filename=package://sherpa_spatial_relations/meshes/hokuyo.dae
