Commit message: added stuff

File: urdf/tree-1.urdf (robot description, URDF)
Before this commit: robot tree1, 1 links, 0 joints
Links:
- link base_link: geometry collision mesh filename=package://sherpa_spatial_relations/meshes/tree-1.stl; visual mesh filename=package://sherpa_spatial_relations/meshes/tree-1.dae
